File: design/main_board/main_board.kicad_pcb (KiCad board)
At the start: 0 parts

Commit message: Finished board layout
Parts:
- added J1: Conn_01x04_Male, Connector_JST:JST_SH_SM04B-SRSS-TB_1x04-1MP_P1.00mm_Horizontal, F.Cu at (162.6, 87.6)
- added J2: Conn_01x04_Male, Connector_JST:JST_SH_SM04B-SRSS-TB_1x04-1MP_P1.00mm_Horizontal, F.Cu at (162.6, 78.7)
- added J3: Conn_01x06_Male, Connector_JST:JST_SH_SM06B-SRSS-TB_1x06-1MP_P1.00mm_Horizontal, F.Cu at (162.6, 97.8)
- added J4: Screw_Terminal_01x02, TerminalBlock_Phoenix:TerminalBlock_Phoenix_MKDS-1,5-2-5.08_1x02_P5.08mm_Horizontal, F.Cu at (161.3, 135.9)
- added J5: Conn_01x04_Male, Connector_JST:JST_SH_SM04B-SRSS-TB_1x04-1MP_P1.00mm_Horizontal, F.Cu at (152.4, 77.5)
- added M1: Fan, TerminalBlock_Phoenix:TerminalBlock_Phoenix_MKDS-1,5-2-5.08_1x02_P5.08mm_Horizontal, F.Cu at (161.3, 113.0)
- added Q1: PSMN6R0-25YLB,115, Package_TO_SOT_SMD:LFPAK56, F.Cu at (149.9, 113.0)
- added Q2: PSMN6R0-25YLB,115, Package_TO_SOT_SMD:LFPAK56, F.Cu at (149.7, 99.1)
- added Q3: PSMN6R0-25YLB,115, Package_TO_SOT_SMD:LFPAK56, F.Cu at (149.9, 124.5)
- added R1: Heater, TerminalBlock_Phoenix:TerminalBlock_Phoenix_MKDS-1,5-2-5.08_1x02_P5.08mm_Horizontal, F.Cu at (161.3, 124.5)
- added R2: 10k, Resistor_SMD:R_0603_1608Metric, F.Cu at (156.2, 83.8)
- added R3: 10k, Resistor_SMD:R_0603_1608Metric, F.Cu at (152.4, 83.8)
- added R4: 10k, Resistor_SMD:R_0603_1608Metric, F.Cu at (147.8, 82.8)
- added U1: NodeMCU_1.0_(ESP-12E), Custom:NodeMCU1.0(12-E), F.Cu at (124.5, 97.8)
- added U2: MC7806BD2TR4G, Custom:MC7806BD2TR4G, F.Cu at (124.8, 130.8)
Routing:
- net +6V: track 0.00 -> 91.7 mm, vias 0 -> 2
- net /BTN_ENC_2: track 0.00 -> 54.6 mm, vias 0 -> 2
- net +12V: track 0.00 -> 51.3 mm
- net /BTN_ENC_1: track 0.00 -> 50.5 mm, vias 0 -> 2
- net /SCL: track 0.00 -> 37.6 mm, vias 0 -> 4
- net /BTN: track 0.00 -> 36.1 mm, vias 0 -> 1
- net /SDA: track 0.00 -> 35.2 mm, vias 0 -> 4
- net /H_CTRL: track 0.00 -> 30.2 mm
- net /ENC_2: track 0.00 -> 27.5 mm, vias 0 -> 2
- net /ENC_1: track 0.00 -> 27.5 mm, vias 0 -> 2
- net /F_CTRL: track 0.00 -> 21.3 mm
- net Net-(Q3-Pad5): track 0.00 -> 13.1 mm
- net Net-(M1-Pad2): track 0.00 -> 13.1 mm
- net Net-(J3-Pad5): track 0.00 -> 11.9 mm
- net GND: track 0.00 -> 11.7 mm, vias 0 -> 74
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- added copper zone on F.Cu, net +12V
- added copper zone on F.Cu, net +3V3
- added copper zone on B.Cu, net GND
- added copper zone on F.Cu, net GND
Other:
- board outline added: 58.4 x 67.3 mm
- copper layers 0 -> 2
- board text added: "Incubator Shake V0.1 Maximilian Schommer"
