File: design/main_board/main_board.kicad_sch (KiCad schematic)
At the start: 10 parts

Commit message: Finished board layout
Parts:
- added J5: Conn_01x04_Male, Connector_JST:JST_SH_SM04B-SRSS-TB_1x04-1MP_P1.00mm_Horizontal, symbol Connector:Conn_01x04_Male
- added R2, R3, R4: 10k, Resistor_SMD:R_0603_1608Metric, symbol Device:R
- added U2: MC7806BD2TR4G, Custom:MC7806BD2TR4G, symbol Custom:MC7806BD2TR4G
- J1, J2: renamed from J?; footprint (none) -> Connector_JST:JST_SH_SM04B-SRSS-TB_1x04-1MP_P1.00mm_Horizontal; MFG_PN (none) -> SM04B-SRSS-TB(LF)(SN); URL (none) -> https://www.adafruit.com/product/4208
- J3: renamed from J?; footprint (none) -> Connector_JST:JST_SH_SM06B-SRSS-TB_1x06-1MP_P1.00mm_Horizontal; MFG_PN (none) -> SM06B-SRSS-TB(LF)(SN); URL (none) -> https://www.digikey.com/en/products/detail/jst-sales-americ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
- J4: renamed from J?; footprint (none) -> TerminalBlock_Phoenix:TerminalBlock_Phoenix_MKDS-1,5-2-5.08_1x02_P5.08mm_Horizontal; MFG_PN (none) -> 1715721; URL (none) -> https://www.digikey.com/en/products/detail/phoenix-contact/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
- M1: renamed from M?; footprint (none) -> TerminalBlock_Phoenix:TerminalBlock_Phoenix_MKDS-1,5-2-5.08_1x02_P5.08mm_Horizontal; MFG_PN (none) -> 1715721; URL (none) -> https://www.digikey.com/en/products/detail/phoenix-contact/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
- Q1, Q2, Q3: renamed from Q?; MFG_PN (none) -> PSMN6R0-25YLB-115; URL (none) -> https://www.digikey.com/en/products/detail/nexperia-usa-inc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
- R1: renamed from R?; footprint (none) -> TerminalBlock_Phoenix:TerminalBlock_Phoenix_MKDS-1,5-2-5.08_1x02_P5.08mm_Horizontal; MFG_PN (none) -> 1715721; URL (none) -> https://www.digikey.com/en/products/detail/phoenix-contact/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
- U1: renamed from U?; footprint (none) -> Custom:NodeMCU1.0(12-E); URL (none) -> https://www.amazon.com/dp/B081CSJV2V
Connections:
- net +12V: now also U2.1 (IN)
- net +3V3: now also J1.2 (Pin_2), J2.2 (Pin_2), J3.4 (Pin_4), U1.11 (3.3V), U1.16 (3.3V), U1.25 (3.3V), R2.1, R3.1, R4.1; no longer J1.3 (Pin_3), J2.3 (Pin_3), J3.3 (Pin_3)
- net +6V: now also J3.6 (Pin_6), U1.15 (VIN), U2.3 (OUT); no longer J3.1 (Pin_1)
- net ENC_1: now also J3.3 (Pin_3), U1.27 (D3(GPIO0)); no longer J3.4 (Pin_4)
- net ENC_2: now also J3.2 (Pin_2), U1.26 (D4(GPIO2)); no longer J3.5 (Pin_5)
- net F_CTRL: now also U1.22 (D6(GPIO12))
- net GND: now also J1.1 (Pin_1), J2.1 (Pin_1), J3.1 (Pin_1), U1.10 (GND), U1.14 (GND), U1.17 (GND), U1.24 (GND), J5.4 (Pin_4), U2.2 (GND); no longer J1.4 (Pin_4), J2.4 (Pin_4), J3.6 (Pin_6)
- net H_CTRL: now also U1.21 (D7(GPIO13))
- net M_CTRL: now also U1.23 (D5(GPIO14))
- net SCL: now also J1.4 (Pin_4), J2.4 (Pin_4), U1.29 (D1(GPIO5)); no longer J1.1 (Pin_1), J2.1 (Pin_1)
- net SDA: now also J1.3 (Pin_3), J2.3 (Pin_3), U1.28 (D2(GPIO4)); no longer J1.2 (Pin_2), J2.2 (Pin_2)
- net at Q2.5 (D): now also J3.5 (Pin_5); no longer J3.2 (Pin_2)
- net BTN: now reaches U1.20 (D8(GPIO15))
- net BTN: now also J5.1 (Pin_1), R2.2
- net BTN_ENC_1: now reaches U1.4 (SD3(GPIO10))
- net BTN_ENC_1: now also J5.3 (Pin_3), R4.2
- net BTN_ENC_2: now reaches U1.5 (SD2(GPIO9))
- net BTN_ENC_2: now also J5.2 (Pin_2), R3.2
- no-connect marks 0 -> 12
Other:
- note added: "BTN"
- note added: "Button and Encoder"
- note added: "ENC_1"
- note added: "ENC_2"
- moved on the sheet: J1, J2, J3, M1, Q1, Q2, Q3, R1
